Commit message: fix(description): turn the body round and give the left wheels their own hand
Two corrections from looking at the machine next to the screen.

The body was 180 degrees out: at body_yaw_deg 90 the model drove backwards, so
the default is 270. That last 180 was never readable from the geometry -- the
files fix the fore-aft AXIS, and nothing in them says which end is the front.

And the left pair needed the opposite hand. Mecanum wheels are chiral, a base
takes two of each, and one was exported; all four were being drawn from it.
mesh_simplify gains a mirror option that reflects about the mesh's own centre
plane, which leaves the bounding box centre alone so the placement offsets
worked out for the original still apply.

It also reverses the winding, which is the point of writing a file rather than
putting a negative <mesh scale> in the URDF: a negative scale reflects the
geometry and leaves the winding, so every face ends up wound backwards and the
wheel renders inside out. Measured on the real wheel -- 65.9% of faces outward
before, 65.9% after mirroring with the correction, 34.1% without it, an exact
complement.

Which hand belongs on which side is the operator's call from looking at the
machine, not something the files could settle, and it says nothing about
roller_layout -- still 'unknown' in supervisor.yaml. This is what the wheels
LOOK like, not a claim about which way they drive.

The URDF also lost another run of two hyphens inside an XML comment, which is
not allowed and had already bitten once. The fix now sweeps for them.

Co-Authored-By: Claude Opus 5 (1M context) <noreply@anthropic.com>

File: src/mdrobot_description/urdf/mdrobot.urdf.xacro (robot description, xacro)
@@ -73,8 +73,15 @@
   <xacro:arg name="body_mesh" default="package://mdrobot_description/meshes/body.stl"/>
   <xacro:arg name="wheel_mesh" default="package://mdrobot_description/meshes/wheel.stl"/>
+  <!-- Mecanum wheels are chiral and only one hand was exported, so the left
+       pair uses a reflection of it: mesh_simplify with its mirror option on z, which flips the
+       roller hand and reverses the winding so the surface still faces out. A
+       negative <mesh scale> would reflect the geometry and leave the winding,
+       and the wheel would render inside out. -->
+  <xacro:arg name="wheel_mesh_left"
+             default="package://mdrobot_description/meshes/wheel_mirror.stl"/>
   <xacro:arg name="mesh_scale" default="0.001 0.001 0.001"/>
   <!-- Rotation about ROS z applied AFTER standing the CAD frame up. See the
        note above: settled by driving the machine, not by reading the files. -->
-  <xacro:arg name="body_yaw_deg" default="90"/>
+  <xacro:arg name="body_yaw_deg" default="270"/>
   <xacro:arg name="wheel_yaw_deg" default="0"/>
   <xacro:property name="body_yaw" value="${radians($(arg body_yaw_deg))}"/>
@@ -82,4 +89,5 @@
   <xacro:property name="body_mesh" value="$(arg body_mesh)"/>
   <xacro:property name="wheel_mesh" value="$(arg wheel_mesh)"/>
+  <xacro:property name="wheel_mesh_left" value="$(arg wheel_mesh_left)"/>
   <!-- Assembly-coordinate offsets, in metres, from mesh_check. -->
   <xacro:property name="body_cx" value="0.256714"/>
@@ -121,8 +129,8 @@
     </visual>
   </link>
-  <xacro:macro name="wheel" params="name x y">
+  <xacro:macro name="wheel" params="name x y mesh">
     <link name="${name}_wheel">
       <visual>
-        <xacro:if value="${wheel_mesh == ''}">
+        <xacro:if value="${mesh == ''}">
           <!-- Cylinders are built along z; the axle runs along y. -->
           <origin rpy="${pi/2} 0 0"/>
@@ -131,12 +139,12 @@
           </geometry>
         </xacro:if>
-        <xacro:unless value="${wheel_mesh == ''}">
+        <xacro:unless value="${mesh == ''}">
           <!-- Same Rx(+90), then the mesh's own bbox centre subtracted so the
                axle sits on the joint. Get this wrong and the wheel orbits.
-               NOTE: mecanum wheels are chiral and only one was supplied, so all
-               four are drawn with the same handedness. roller_layout is
-               'unknown' on this machine anyway — which way the rollers face has
-               never been settled, and drawing a specific one would be asserting
-               something nobody has checked. -->
+               The left pair gets the mirrored mesh: which hand goes where is
+               the operator's call, made by looking at the machine, not
+               something the files could settle. roller_layout is still
+               'unknown' in supervisor.yaml, so this is what the wheels LOOK
+               like and not a claim about which way the rollers drive. -->
           <origin rpy="${pi/2} 0 ${wheel_yaw}"
                   xyz="${-(wheel_cx*cos(wheel_yaw) + wheel_cz*sin(wheel_yaw))}
@@ -144,5 +152,5 @@
                        ${-wheel_cy}"/>
           <geometry>
-            <mesh filename="${wheel_mesh}" scale="$(arg mesh_scale)"/>
+            <mesh filename="${mesh}" scale="$(arg mesh_scale)"/>
           </geometry>
         </xacro:unless>
@@ -159,8 +167,8 @@
   <!-- Joint names are the WHEEL_NAMES the whole workspace uses. Rename one and
        robot_state_publisher silently stops turning that wheel. -->
-  <xacro:wheel name="front_left"  x="${ wheelbase/2}" y="${ track/2}"/>
-  <xacro:wheel name="front_right" x="${ wheelbase/2}" y="${-track/2}"/>
-  <xacro:wheel name="rear_left"   x="${-wheelbase/2}" y="${ track/2}"/>
-  <xacro:wheel name="rear_right"  x="${-wheelbase/2}" y="${-track/2}"/>
+  <xacro:wheel name="front_left"  x="${ wheelbase/2}" y="${ track/2}" mesh="${wheel_mesh_left}"/>
+  <xacro:wheel name="front_right" x="${ wheelbase/2}" y="${-track/2}" mesh="${wheel_mesh}"/>
+  <xacro:wheel name="rear_left"   x="${-wheelbase/2}" y="${ track/2}" mesh="${wheel_mesh_left}"/>
+  <xacro:wheel name="rear_right"  x="${-wheelbase/2}" y="${-track/2}" mesh="${wheel_mesh}"/>
   <!-- Where the HWT901B is bolted. The offset is a GUESS — nothing reads it
        yet, because the heading is used as a change from a reference and a lever

Commit message: fix(description): the mirror belonged on the right pair
Put on the left, corrected by looking at the machine. Which hand goes where
was never readable from the files -- both are geometrically valid bases -- so
this was always going to take one look and possibly one correction.

What made the correction cost a round trip was the naming. The two arguments
were "wheel_mesh" and "wheel_mesh_left", so the first said nothing about which
side it was for and the pair gave no way to see at a glance which pair had the
reflection. They are wheel_mesh_left and wheel_mesh_right now, and the URDF
prints which corner takes which.

Co-Authored-By: Claude Opus 5 (1M context) <noreply@anthropic.com>

File: src/mdrobot_description/urdf/mdrobot.urdf.xacro (robot description, xacro)
@@ -72,11 +72,16 @@
   <xacro:property name="body_height" value="0.189"/>
   <xacro:arg name="body_mesh" default="package://mdrobot_description/meshes/body.stl"/>
-  <xacro:arg name="wheel_mesh" default="package://mdrobot_description/meshes/wheel.stl"/>
-  <!-- Mecanum wheels are chiral and only one hand was exported, so the left
-       pair uses a reflection of it: mesh_simplify with its mirror option on z, which flips the
-       roller hand and reverses the winding so the surface still faces out. A
-       negative <mesh scale> would reflect the geometry and leave the winding,
-       and the wheel would render inside out. -->
+  <!-- Mecanum wheels are chiral and only one hand was exported, so one side
+       is a reflection of it: mesh_simplify with its mirror option on z, which
+       flips the roller hand and reverses the winding so the surface still
+       faces out. A negative <mesh scale> would reflect the geometry and leave
+       the winding alone, and that wheel would render inside out.
+       WHICH side takes the mirror was settled by looking at the machine: it is
+       the RIGHT pair. Named by side rather than "the mesh" and "the other
+       one", because the first attempt put it on the wrong pair and the names
+       gave no way to notice. -->
   <xacro:arg name="wheel_mesh_left"
+             default="package://mdrobot_description/meshes/wheel.stl"/>
+  <xacro:arg name="wheel_mesh_right"
              default="package://mdrobot_description/meshes/wheel_mirror.stl"/>
   <xacro:arg name="mesh_scale" default="0.001 0.001 0.001"/>
@@ -88,6 +93,6 @@
   <xacro:property name="wheel_yaw" value="${radians($(arg wheel_yaw_deg))}"/>
   <xacro:property name="body_mesh" value="$(arg body_mesh)"/>
-  <xacro:property name="wheel_mesh" value="$(arg wheel_mesh)"/>
   <xacro:property name="wheel_mesh_left" value="$(arg wheel_mesh_left)"/>
+  <xacro:property name="wheel_mesh_right" value="$(arg wheel_mesh_right)"/>
   <!-- Assembly-coordinate offsets, in metres, from mesh_check. -->
   <xacro:property name="body_cx" value="0.256714"/>
@@ -142,5 +147,5 @@
           <!-- Same Rx(+90), then the mesh's own bbox centre subtracted so the
                axle sits on the joint. Get this wrong and the wheel orbits.
-               The left pair gets the mirrored mesh: which hand goes where is
+               The RIGHT pair gets the mirrored mesh: which hand goes where is
                the operator's call, made by looking at the machine, not
                something the files could settle. roller_layout is still
@@ -168,7 +173,7 @@
        robot_state_publisher silently stops turning that wheel. -->
   <xacro:wheel name="front_left"  x="${ wheelbase/2}" y="${ track/2}" mesh="${wheel_mesh_left}"/>
-  <xacro:wheel name="front_right" x="${ wheelbase/2}" y="${-track/2}" mesh="${wheel_mesh}"/>
+  <xacro:wheel name="front_right" x="${ wheelbase/2}" y="${-track/2}" mesh="${wheel_mesh_right}"/>
   <xacro:wheel name="rear_left"   x="${-wheelbase/2}" y="${ track/2}" mesh="${wheel_mesh_left}"/>
-  <xacro:wheel name="rear_right"  x="${-wheelbase/2}" y="${-track/2}" mesh="${wheel_mesh}"/>
+  <xacro:wheel name="rear_right"  x="${-wheelbase/2}" y="${-track/2}" mesh="${wheel_mesh_right}"/>
   <!-- Where the HWT901B is bolted. The offset is a GUESS — nothing reads it
        yet, because the heading is used as a change from a reference and a lever
